File: pcb/pmod_d_mikroshield.kicad_sch (KiCad schematic)
At the start: 7 parts, among them J1 CON_HDR_MIKROBUS_ADDON_TH, J2 CON_HDR_100MILS_F_TH_RA_2X6, J3 CON_HDR_100MILS_M_TH_1X3, J4 CON_HDR_100MILS_M_TH_1X2, J5 CON_HDR_100MILS_M_TH_1X2

Commit message: Silkscreen fixes
Other:
- note added: "Voltage jumper"
- note removed: "Voltage header"
Changed lines of the file:
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@@
     (stroke (width 0) (type default) (color 0 0 0 0))
   )
-  (text "Voltage header" (at 105.41 20.32 0)
+  (text "Voltage jumper" (at 105.41 20.32 0)
     (effects (font (size 2.54 2.54)) (justify left bottom))
   )
